File: IOexpanderModule.brd (EAGLE design)
At the start: 51.3 x 64 mm, 32 parts, among them J2 4P-3.5mm-TERMINAL, J3 4P-3.5MM-TERMINAL, J4 SDA, J5 GND, J6 3V3, J7 SCL, U1 PCF8574DW

Commit message: CAM and CAD files added
Parts:
- J2: value 4P-3.5mm-TERMINAL -> 4P-3.5MM-TERMINAL
Routing:
- net F2+: track 18.4 -> 19.0 mm
